File: audiomute.kicad_sch (KiCad schematic)
At the start: 20 parts, among them J1 SJ-3524-SMT, J2 B2B-XH-A_LF__SN_, J3 B2B-XH-A_LF__SN_, J4 SJ-3524-SMT, Q1 NPN, Q2 PNP, Q3 NPN, Q4 NPN, U1 J104D2C5VDC.20S

Commit message: Minor update to notes in schematic.
Other:
- note added: "The mute signal comes from the controller. This signal goes high during auto-tune, thus muting the audio to prevent an annoying tone in the receiver output."
- note removed: "Mute when +5V, audio passes through 0V."
- note removed: "This is be the same signal as the controller op-amp supply."
Changed lines of the file:
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@@
     (effects (font (size 2 2) (thickness 0.4) bold) (justify left bottom))
-  )
-  (text "Mute when +5V, audio passes through 0V." (at 52.07 119.38 0)
-    (effects (font (size 1.27 1.27) bold) (justify left bottom))
   )
   (text "Output Line Audio or Speaker" (at 204.47 58.42 0)
@@
     (effects (font (size 2 2) (thickness 0.4) bold) (justify left bottom))
   )
-  (text "This is be the same signal as\nthe controller op-amp supply."
-    (at 52.07 124.46 0)
+  (text "The mute signal comes from the controller.\nThis signal goes high during auto-tune,\nthus muting the audio to prevent an annoying\ntone in the receiver output."
+    (at 49.53 125.73 0)
     (effects (font (size 1.27 1.27) bold) (justify left bottom))
   )
